Commit message: Better drone model (from @gstavrinos) with fixed orientation (in urdf), updated geometric calibration for bebop2

File: bebop_description/urdf/bebop_base.urdf.xacro (robot description, xacro)
@@ -14,6 +14,7 @@
   <link name="base_link">
    <visual>
+      <origin rpy="0 0 1.57075"/>
       <geometry>
-        <mesh scale=".001 .001 .001" filename="package://bebop_description/meshes/bebop_model.stl"/>
+        <mesh filename="package://bebop_description/meshes/bebop_model.stl"/>
       </geometry>
    </visual>
